File: v2_00-0a/hardware/rpi_cm4_cm5_CarrierBoard/CM4_CM5_CONN_A.kicad_sch (KiCad schematic)
At the start: 69 parts, among them J19 RPI_CMx_A, J6 M20-9990245, J7 2998TR, Q12 2N7002, U19 SN74LVC1G125DBVR, U20 SN74LVC1G07DBVR, U21 MCP7940NT-I/MS, U5 SN74LVC1G125DBVR, Y2 32.768kHz

Commit message: Add and modify existing schematics
Other:
- note added: "Resistors are 1% 1/16W 0402 unless otherwise noted Capacitors are 10% 50V X7R 0402 unless otherwise noted"
- moved on the sheet: R156
Changed lines of the file:
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@@
 		)
 	)
+	(text "Resistors are 1% 1/16W 0402 unless otherwise noted\nCapacitors are 10% 50V X7R 0402 unless otherwise noted"
+		(exclude_from_sim no)
+		(at 12.7 170.942 0)
+		(effects
+			(font
+				(size 1.27 1.27)
+			)
+			(justify left)
+		)
+	)
 	(text "HW watchdog"
 		(exclude_from_sim no)
@@
 	)
 	(junction
-		(at 103.505 176.53)
+		(at 104.775 176.53)
 		(diameter 0)
 		(color 0 0 0 0)
@@
 	(wire
 		(pts
-			(xy 103.505 166.37) (xy 103.505 168.91)
+			(xy 104.775 166.37) (xy 104.775 168.91)
 		)
 		(stroke
@@
 	(wire
 		(pts
-			(xy 103.505 175.26) (xy 103.505 176.53)
+			(xy 104.775 175.26) (xy 104.775 176.53)
 		)
 		(stroke
@@
 	(wire
 		(pts
+			(xy 104.775 176.53) (xy 106.68 176.53)
+		)
+		(stroke
+			(width 0)
+			(type default)
+		)
+	)
+	(wire
+		(pts
 			(xy 214.63 27.94) (xy 214.63 29.21)
 		)
@@
 	(wire
 		(pts
-			(xy 81.915 176.53) (xy 103.505 176.53)
+			(xy 81.915 176.53) (xy 104.775 176.53)
 		)
 		(stroke
@@
 		)
 	)
-	(wire
-		(pts
-			(xy 103.505 176.53) (xy 106.68 176.53)
-		)
-		(stroke
-			(width 0)
-			(type default)
-		)
-	)
 	(bus
 		(pts
@@
 	(symbol
 		(lib_id "KiCad_Pwr_Symbols:+1V8")
-		(at 103.505 166.37 0)
+		(at 104.775 166.37 0)
 		(unit 1)
 		(exclude_from_sim no)
@@
 		(dnp no)
 		(property "Reference" "#PWR0203"
-			(at 103.505 170.18 0)
+			(at 104.775 170.18 0)
 			(effects
 				(font
@@
 		)
 		(property "Value" "5V0_CB"
-			(at 103.505 162.56 0)
+			(at 104.775 162.56 0)
 			(effects
 				(font
@@
 		)
 		(property "Footprint" ""
-			(at 103.505 166.37 0)
+			(at 104.775 166.37 0)
 			(effects
 				(font
@@
 		)
 		(property "Datasheet" ""
-			(at 103.505 166.37 0)
+			(at 104.775 166.37 0)
 			(effects
 				(font
@@
 		)
 		(property "Description" "Power symbol creates a global label with name \"+1V8\""
-			(at 103.505 166.37 0)
+			(at 104.775 166.37 0)
 			(effects
 				(font
@@
 	(symbol
 		(lib_id "KicadCompDb:Resistors/RES_SMT_00020")
-		(at 103.505 173.99 90)
+		(at 104.775 173.99 90)
 		(unit 1)
 		(exclude_from_sim no)
@@
 		(dnp no)
 		(property "Reference" "R156"
-			(at 104.394 170.942 90)
+			(at 105.664 170.942 90)
 			(effects
 				(font
@@
 		)
 		(property "Value" "510K"
-			(at 104.394 173.482 90)
+			(at 105.664 173.482 90)
 			(effects
 				(font
@@
 		)
 		(property "Footprint" "footprint:RES_0402"
-			(at 125.603 173.482 0)
+			(at 126.873 173.482 0)
 			(effects
 				(font
@@
 		)
 		(property "Datasheet" "https://www.yageogroup.com/content/datasheet/asset/file/PYU-RC_GROUP_51_ROHS_L"
-			(at 103.505 173.99 0)
+			(at 104.775 173.99 0)
 			(effects
 				(font
@@
 		)
 		(property "Description" "RES 510K OHM 1% 1/16W 0402"
-			(at 113.411 172.212 0)
+			(at 114.681 172.212 0)
 			(effects
 				(font
@@
 		)
 		(property "Tolerance" "1%"
-			(at 123.825 173.736 0)
+			(at 125.095 173.736 0)
 			(effects
 				(font
@@
 		)
 		(property "Power" "1/16W"
-			(at 117.729 173.736 0)
+			(at 118.999 173.736 0)
 			(effects
 				(font
@@
 		)
 		(property "Package" "0402"
-			(at 119.761 173.99 0)
+			(at 121.031 173.99 0)
 			(effects
 				(font
@@
 		)
 		(property "Manufacturer" "YAGEO"
-			(at 121.793 173.736 0)
+			(at 123.063 173.736 0)
 			(effects
 				(font
@@
 		)
 		(property "Manufacturer Part Number" "RC0402FR-10510KL"
-			(at 111.379 173.736 0)
+			(at 112.649 173.736 0)
 			(effects
 				(font
@@
 		)
 		(property "Distributor" "DigiKey"
-			(at 109.347 173.99 0)
+			(at 110.617 173.99 0)
 			(effects
 				(font
@@
 		)
 		(property "Distributor Part Number" "13-RC0402FR-10510KLCT-ND"
-			(at 115.697 173.228 0)
+			(at 116.967 173.228 0)
 			(effects
 				(font
@@
 		)
 		(property "Temperature Coefficient" "±100ppm/°C"
-			(at 103.505 173.99 0)
+			(at 104.775 173.99 0)
 			(effects
 				(font
@@
 		)
 		(property "Operating Temperature" "-55°C ~ 155°C"
-			(at 127.889 173.228 0)
+			(at 129.159 173.228 0)
 			(effects
 				(font
@@
 		)
 		(property "Type" "RES SMT"
-			(at 103.505 173.99 0)
+			(at 104.775 173.99 0)
 			(show_name yes)
 			(effects
@@
 		)
 		(property "Dimensions" "1.00mm x 0.50mm"
-			(at 103.505 173.99 0)
+			(at 104.775 173.99 0)
 			(show_name yes)
 			(effects
