File: v2_00-0a/hardware/rpi_cm4_cm5_CarrierBoard/RESET_SUPERVISOR.kicad_sch (KiCad schematic)
At the start: 21 parts, among them Q1 2N7002, Q2 2N7002, Q3 2N7002, U1 STM6710DWB6F, U2 SN74LVC1G125DBVR, U3 SN74LVC1G125DBVR

Commit message: Add and modify existing schematics
Connections:
- net 1V0_CB renamed 1V05_CB
Other:
- moved on the sheet: C1, C2, C3, C4, C5, C6, D1, Q1, Q2, Q3, R1, R2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
