File: v2_00-0a/hardware/rpi_cm4_cm5_CarrierBoard/TFT_CONN.kicad_sch (KiCad schematic)
At the start: 20 parts, among them J8 62684-402100ALF, J9 5051101092

Commit message: Add and modify existing schematics
Other:
- note added: "Resistors are 1% 1/16W 0402 unless otherwise noted Capacitors are 10% 50V X7R 0402 unless otherwise noted"
- moved on the sheet: C124, C125, D21, D22, D23, J8, J9
