File: v2_00-0a/hardware/rpi_cm4_cm5_CarrierBoard/TFT_POWER.kicad_sch (KiCad schematic)
At the start: 67 parts, among them Q14 2N7002, Q15 2N7002, Q16 BCP56-16, Q17 ISP75DP06LMXTSA1, Q18 MMBT3904-7-F, U24 MAX16928CGUP, U25 TPS79901DRVR, U26 TPS61169DCKR, U27 AP22913W6-7

Commit message: Update schematic
Parts:
- added C156, C159, C162, C163, C165, C166: 22u, footprint:CAP_NONPOL_0805, symbol KicadCompDb:Capacitors/CAP_CER_SMT_00011
- added C157: 100p, footprint:CAP_NONPOL_0402, symbol KicadCompDb:Capacitors/CAP_CER_SMT_00007
- added C158, C160, C161, C164: 0.1u, footprint:CAP_NONPOL_0402, symbol KicadCompDb:Capacitors/CAP_CER_SMT_00001
- added D30: SK34A-LTP, footprint:DO-214AC, symbol KicadCompDb:Diodes/DIODE_00005
- added L5: PA5003.472NLT, footprint:PA5003, symbol KicadCompDb:Inductor/IND_00008
- added R206: 4K7, footprint:RES_0402, symbol KicadCompDb:Resistors/RES_SMT_00010
- added R207: 2K2, footprint:RES_0402, symbol KicadCompDb:Resistors/RES_SMT_00008
- added R208: 10K, footprint:RES_0402, symbol KicadCompDb:Resistors/RES_SMT_00013
- added R209, R210: 1R5, footprint:RES_0603, symbol KicadCompDb:Resistors/RES_SMT_00007
- added R211: 0R, footprint:RES_1206, symbol KicadCompDb:Resistors/RES_SMT_00022
Connections:
- net 5V0_CB: now also U25.6 (IN), U26.5 (VIN), C156.2, C158.2, C164.2, C165.2, C166.2, L5.1
- net GND: now also U25.3 (GND), U25.7 (EP), U26.2 (GND), C156.1, C158.1, C159.1, C160.1, C161.1, C162.1, C163.1, C164.1, C165.1, C166.1, R207.1, R208.1, R209.1, R210.1
- net TFT_STBYB: now also U25.4 (EN)
- net TFT_3V8: now reaches U25.1 (OUT)
- net TFT_3V8: now also C157.2, C159.2, C160.2, R206.1
- net at U25.2 (FB): now also C157.1, R206.2, R207.2
- net at U26.1 (SW): now also D30.2 (A), L5.2
- net TFT_LED-: now reaches U26.3 (FB)
- net TFT_LED-: now also R209.2, R210.2
- new net: C161.2, C162.2, C163.2, D30.1 (K), R211.1
- new net BL_PWM: R208.2, U26.2 (GND)
- new net TFT_LED+: R211.2
Other:
- note added: "0R for I(meas)"
- moved on the sheet: C126, C127, C128, C129, C130, C131, C132, C133, C134, C135, C136, C137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

Commit message: Add and modify existing schematics
Connections:
- net 5V0_CB: no longer C164.2, C165.2, C166.2, L5.1, U26.5 (VIN)
- net BL_PWM: now also U26.4 (CTRL); no longer U26.2 (GND)
- new net 3V3_CB: C164.2, C165.2, C166.2, L5.1, U26.5 (VIN)
Other:
- note added: "Resistors are 1% 1/16W 0402 unless otherwise noted Capacitors are 10% 50V X7R 0402 unless otherwise noted"
Changed lines of the file:
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@@
 		(comment 8 "WIP")
 	)
+	(text "Resistors are 1% 1/16W 0402 unless otherwise noted\nCapacitors are 10% 50V X7R 0402 unless otherwise noted"
+		(exclude_from_sim no)
+		(at 12.7 170.942 0)
+		(effects
+			(font
+				(size 1.27 1.27)
+			)
+			(justify left)
+		)
+	)
 	(text "TFT Charge Pump for\nVGH and VGL rails\n"
 		(exclude_from_sim no)
@@
 		)
 		(property "Current (Rated)" "5.9A"
-			(at 151.638 17.018 0)
+			(at 154.94 17.018 0)
 			(effects
 				(font
@@
 		)
 		(property "Inductance" "4.7uH"
-			(at 149.86 15.875 0)
-			(show_name yes)
+			(at 149.606 17.018 0)
 			(effects
 				(font
 					(size 1.27 1.27)
 				)
-				(hide yes)
 			)
 		)
@@
 		(pin "5"
 		)
-		(pin "2"
+		(pin "4"
 		)
 		(pin "3"
@@
 			)
 		)
-		(property "Value" "5V0_CB"
+		(property "Value" "3V3_CB"
 			(at 112.903 16.129 0)
 			(effects
