File: v2_00-0a/hardware/rpi_cm4_cm5_CarrierBoard/USB_MUX.kicad_sch (KiCad schematic)
At the start: 5 parts, among them U22 FSUSB42UMX

Commit message: Add and modify existing schematics
Other:
- note added: "Resistors are 1% 1/16W 0402 unless otherwise noted Capacitors are 10% 50V X7R 0402 unless otherwise noted"
Changed lines of the file:
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@@
 		(comment 8 "WIP")
+	)
+	(text "Resistors are 1% 1/16W 0402 unless otherwise noted\nCapacitors are 10% 50V X7R 0402 unless otherwise noted"
+		(exclude_from_sim no)
+		(at 12.7 170.942 0)
+		(effects
+			(font
+				(size 1.27 1.27)
+			)
+			(justify left)
+		)
 	)
 	(junction
@@
 		(on_board yes)
 		(dnp no)
-		(fields_autoplaced yes)
 		(property "Reference" "U22"
-			(at 147.32 72.39 0)
+			(at 147.32 76.454 0)
 			(effects
 				(font
@@
 		)
 		(property "Value" "FSUSB42UMX"
-			(at 147.32 74.93 0)
-			(effects
-				(font
+			(at 147.066 94.996 0)
+			(effects
+				(font
