File: v2_00-0a/hardware/rpi_cm4_cm5_CarrierBoard/rpi_cm4_cm5_CarrierBoard.kicad_pcb (KiCad board)
At the start: 2 copper layers, 181.6 x 100.6 mm, 366 parts, among them J1 DM3AT-SF-PEJM5, J19 RPI_CMx_A, J2 0484050003, J3 0484050003, J4 2086581001, J5 0826-1X1T-32-F, J6 M20-9990245, J7 2998TR, Q1 2N7002, Q10 SSM3K56FS,LF, Q11 SSM3K56FS,LF, Q12 2N7002, Q2 2N7002, Q3 2N7002, Q4 2N7002, Q5 2N7002, Q6 2N7002, Q7 2N7002, Q8 2N7002, U1 STM6710DWB6F, U10 TLV62130ARGTR, U11 TLV62130ARGTR, U12 TPS7A7002DDAR, U13 SE555DR, U14 SN74LVC1G14DBVR, U15 SN65DSI84ZXHR, U16 SN74LVC1G125DBVR, U17 RPI_CMx_B, U18 AP22913W6-7, U19 SN74LVC1G125DBVR, U2 SN74LVC1G125DBVR, U20 SN74LVC1G07DBVR, U21 MCP7940NT-I/MS, U3 SN74LVC1G125DBVR, U4 AP22913W6-7, U5 SN74LVC1G125DBVR, U6 SST25VF512A, U7 UPD720202K8-711-BAA-A, U8 AP2192AFGEG-7, U9 TLV62130ARGTR, Y1 24MHz, Y2 32.768kHz

Commit message: Add and modify existing schematics
Parts:
- removed R76: 8K06, footprint:RES_0402
- removed R78: 10K, footprint:RES_0402
- added C110: 0.1u, footprint:CAP_NONPOL_0402, F.Cu at (215.7, 128.6)
- added C112: 0.1u, footprint:CAP_NONPOL_0402, F.Cu at (215.7, 130.7)
- added C114: 22u, footprint:CAP_NONPOL_0805, F.Cu at (124.7, 141.3)
- added C117: 22u, footprint:CAP_NONPOL_0805, F.Cu at (124.7, 144.2)
- added C119: 22u, footprint:CAP_NONPOL_0805, F.Cu at (124.7, 147.1)
- added C120: 22u, footprint:CAP_NONPOL_0805, F.Cu at (124.7, 150.0)
- added C121: 22u, footprint:CAP_NONPOL_0805, F.Cu at (124.7, 152.9)
- added C122: 0.1u, footprint:CAP_NONPOL_0402, F.Cu at (135.8, 140.9)
- added C123: 0.1u, footprint:CAP_NONPOL_0402, F.Cu at (141.0, 146.1)
- added C124: 1u, footprint:CAP_NONPOL_0805, F.Cu at (104.3, 153.6)
- added C125: 0.1u, footprint:CAP_NONPOL_0402, F.Cu at (107.8, 153.2)
- added C126: 22u, footprint:CAP_NONPOL_0805, F.Cu at (36.9, 89.3)
- added C127: 22u, footprint:CAP_NONPOL_0805, F.Cu at (36.9, 92.2)
- added C128: 0.1u, footprint:CAP_NONPOL_0402, F.Cu at (21.4, 88.9)
- added C129: 0.1u, footprint:CAP_NONPOL_0402, F.Cu at (21.4, 91.0)
- added C130: 0.1u, footprint:CAP_NONPOL_0402, F.Cu at (21.4, 93.1)
- added C131: 22u, footprint:CAP_NONPOL_0805, F.Cu at (36.9, 95.1)
- added C132: 22u, footprint:CAP_NONPOL_0805, F.Cu at (36.9, 98.0)
- added C133: 0.1u, footprint:CAP_NONPOL_0402, F.Cu at (21.4, 95.2)
- added C134: 0.1u, footprint:CAP_NONPOL_0402, F.Cu at (21.4, 97.3)
- added C135: 220p, footprint:CAP_NONPOL_0402, F.Cu at (21.4, 99.4)
- added C136: 22p, footprint:CAP_NONPOL_0402, F.Cu at (21.4, 101.5)
- added C137: 560p, footprint:CAP_NONPOL_0402, F.Cu at (21.4, 103.6)
- added C138: 1u, footprint:CAP_NONPOL_0805, F.Cu at (36.9, 100.9)
- added C139: 1u, footprint:CAP_NONPOL_0805, F.Cu at (36.9, 103.8)
- added C140: 1u, footprint:CAP_NONPOL_0805, F.Cu at (36.9, 106.7)
- added C141: 1u, footprint:CAP_NONPOL_0805, F.Cu at (40.9, 89.3)
- added C142: 0.1u, footprint:CAP_NONPOL_0402, F.Cu at (21.4, 105.7)
- added C143: 0.1u, footprint:CAP_NONPOL_0402, F.Cu at (21.4, 107.8)
- added C144: 22u, footprint:CAP_NONPOL_0805, F.Cu at (40.9, 92.2)
- added C145: 22u, footprint:CAP_NONPOL_0805, F.Cu at (40.9, 95.1)
- added C146: 0.1u, footprint:CAP_NONPOL_0402, F.Cu at (24.4, 88.9)
- added C147: 22p, footprint:CAP_NONPOL_0402, F.Cu at (24.4, 91.0)
- added C148: 0.1u, footprint:CAP_NONPOL_0402, F.Cu at (24.4, 93.1)
- added C149: 22u, footprint:CAP_NONPOL_0805, F.Cu at (40.9, 98.0)
- added C150: 22u, footprint:CAP_NONPOL_0805, F.Cu at (40.9, 100.9)
- added C151: 22p, footprint:CAP_NONPOL_0402, F.Cu at (24.4, 95.2)
- added C152: 100p, footprint:CAP_NONPOL_0402, F.Cu at (24.4, 97.3)
- added C153: 0.1u, footprint:CAP_NONPOL_0402, F.Cu at (24.4, 99.4)
- added C154: 22u, footprint:CAP_NONPOL_0805, F.Cu at (40.9, 103.8)
- added C155: 0.1u, footprint:CAP_NONPOL_0402, F.Cu at (24.4, 101.5)
- added C156: 22u, footprint:CAP_NONPOL_0805, F.Cu at (40.9, 106.7)
- added C157: 100p, footprint:CAP_NONPOL_0402, F.Cu at (24.4, 103.6)
- added C158: 0.1u, footprint:CAP_NONPOL_0402, F.Cu at (24.4, 105.7)
- added C159: 22u, footprint:CAP_NONPOL_0805, F.Cu at (44.9, 89.3)
- added C160: 0.1u, footprint:CAP_NONPOL_0402, F.Cu at (24.4, 107.8)
- added C161: 0.1u, footprint:CAP_NONPOL_0402, F.Cu at (27.4, 88.9)
- added C162: 22u, footprint:CAP_NONPOL_0805, F.Cu at (44.9, 92.2)
- added C163: 22u, footprint:CAP_NONPOL_0805, F.Cu at (44.9, 95.1)
- added C164: 0.1u, footprint:CAP_NONPOL_0402, F.Cu at (27.4, 91.0)
- added C165: 22u, footprint:CAP_NONPOL_0805, F.Cu at (44.9, 98.0)
- added C166: 22u, footprint:CAP_NONPOL_0805, F.Cu at (44.9, 100.9)
- added C167: 1u, footprint:CAP_NONPOL_0805, F.Cu at (148.9, 154.2)
- added C168: 0.1u, footprint:CAP_NONPOL_0402, F.Cu at (170.9, 122.1)
- added C169: 10n, footprint:CAP_NONPOL_0402, F.Cu at (173.9, 117.9)
- added C170: 10n, footprint:CAP_NONPOL_0402, F.Cu at (173.9, 120.0)
- added C171: 0.1u, footprint:CAP_NONPOL_0402, F.Cu at (173.9, 122.1)
- added D11: SK34A-LTP, footprint:DO-214AC, F.Cu at (119.0, 141.8)
- added D17: MMSZ5242B-TP, footprint:SOD-123, F.Cu at (118.1, 156.9)
- added D18: SK34A-LTP, footprint:DO-214AC, F.Cu at (119.0, 145.7)
- added D19: SML4761A-E3/5A, footprint:DO-214AC, F.Cu at (119.0, 149.6)
- added D20: SK34A-LTP, footprint:DO-214AC, F.Cu at (119.0, 153.5)
- added D21: ESD7016MUTAG, footprint:UDFN8, F.Cu at (104.5, 148.2)
- added D22: ESD7016MUTAG, footprint:UDFN8, F.Cu at (104.5, 150.9)
- added D23: D1213A-02SOL-7, footprint:SOT-23-3, F.Cu at (109.0, 149.0)
- added D24: BAT42WS-TP, footprint:SOD-323, F.Cu at (26.4, 110.2)
- added D25: BAT42WS-TP, footprint:SOD-323, F.Cu at (26.4, 112.9)
- added D26: BAT42WS-TP, footprint:SOD-323, F.Cu at (26.4, 115.7)
- added D27: BAT42WS-TP, footprint:SOD-323, F.Cu at (26.4, 118.4)
- added D28: SK34A-LTP, footprint:DO-214AC, F.Cu at (50.6, 89.8)
- added D29: SK34A-LTP, footprint:DO-214AC, F.Cu at (50.6, 93.7)
- added D30: SK34A-LTP, footprint:DO-214AC, F.Cu at (50.6, 97.6)
- added J8: 62684-402100ALF, footprint:62684-402100ALF, F.Cu at (72.9, 143.9)
- added J9: 5051101092, footprint:5051101092, F.Cu at (104.8, 143.3)
- added L4: SRN8040-100M, footprint:SRN8040, F.Cu at (39.8, 122.7)
- added L5: PA5003.472NLT, footprint:PA5003, F.Cu at (31.5, 111.9)
- added Q13: 2N7002, footprint:SOT-23-3, F.Cu at (144.7, 154.8)
- added Q14: 2N7002, footprint:SOT-23-3, F.Cu at (22.1, 110.9)
- added Q15: 2N7002, footprint:SOT-23-3, F.Cu at (22.1, 115.0)
- added Q16: BCP56-16, footprint:SOT-223-4, F.Cu at (38.9, 113.0)
- added Q17: ISP75DP06LMXTSA1, footprint:SOT-223-4, F.Cu at (46.9, 113.0)
- added Q18: MMBT3904-7-F, footprint:SOT-23-3, F.Cu at (22.1, 119.2)
- added Q9: IPD60R360P7ATMA1, footprint:TO-252-3, F.Cu at (130.5, 146.3)
- added R177: 6K04, footprint:RES_0402, F.Cu at (215.7, 132.8)
- added R178: 10K, footprint:RES_0402, F.Cu at (215.7, 134.9)
- added R179: 1K, footprint:RES_0402, F.Cu at (135.8, 143.0)
- added R180: 1K, footprint:RES_0402, F.Cu at (135.8, 145.1)
- added R181: 470R, footprint:RES_0402, F.Cu at (135.8, 147.2)
- added R182: 22R, footprint:RES_0402, F.Cu at (135.8, 149.3)
- added R183: 0R, footprint:RES_1206, F.Cu at (129.3, 154.3)
- added R184: 0R, footprint:RES_1206, F.Cu at (129.3, 157.9)
- added R185: 10K, footprint:RES_0402, F.Cu at (27.4, 93.1)
- added R186: 10K, footprint:RES_0402, F.Cu at (27.4, 95.2)
- added R187: 10K, footprint:RES_0402, F.Cu at (27.4, 97.3)
- added R188: 30K1, footprint:RES_0402, F.Cu at (27.4, 99.4)
- added R189: 10K, footprint:RES_0402, F.Cu at (27.4, 101.5)
- added R190: 10K, footprint:RES_0402, F.Cu at (27.4, 103.6)
- added R191: 1Meg, footprint:RES_0402, F.Cu at (27.4, 105.7)
- added R192: 10K, footprint:RES_0402, F.Cu at (27.4, 107.8)
- added R193: 34K, footprint:RES_0402, F.Cu at (30.4, 88.9)
- added R194: 169K, footprint:RES_0402, F.Cu at (30.4, 91.0)
- added R195: 10K, footprint:RES_0402, F.Cu at (30.4, 93.1)
- added R196: 10K, footprint:RES_0402, F.Cu at (30.4, 95.2)
- added R197: 86K6, footprint:RES_0402, F.Cu at (30.4, 97.3)
- added R198: 10K, footprint:RES_0402, F.Cu at (30.4, 99.4)
- added R199: 10K, footprint:RES_0402, F.Cu at (30.4, 101.5)
- added R200: 169K, footprint:RES_0402, F.Cu at (30.4, 103.6)
- added R201: 6K81, footprint:RES_0402, F.Cu at (30.4, 105.7)
- added R202: 475K, footprint:RES_0402, F.Cu at (30.4, 107.8)
- added R203: 82K5, footprint:RES_0402, F.Cu at (33.4, 88.9)
- added R204: 6K81, footprint:RES_0402, F.Cu at (33.4, 91.0)
- added R205: 10K, footprint:RES_0402, F.Cu at (33.4, 93.1)
- added R206: 4K7, footprint:RES_0402, F.Cu at (33.4, 95.2)
- added R207: 2K2, footprint:RES_0402, F.Cu at (33.4, 97.3)
- added R208: 10K, footprint:RES_0402, F.Cu at (33.4, 99.4)
- added R209: 1R5, footprint:RES_0603, F.Cu at (30.3, 121.0)
- added R210: 1R5, footprint:RES_0603, F.Cu at (30.3, 123.4)
- added R211: 0R, footprint:RES_1206, F.Cu at (31.2, 116.7)
- added U22: FSUSB42UMX, footprint:10-UMLP, F.Cu at (219.1, 129.3)
- added U23: LTC4359IDCB, footprint:6-WFDFN-EP, F.Cu at (134.5, 154.2)
- added U24: MAX16928CGUP, footprint:TSSOP-20-EP, F.Cu at (49.5, 121.7)
- added U25: TPS79901DRVR, footprint:WSON-6-EP, F.Cu at (26.4, 126.0)
- added U26: TPS61169DCKR, footprint:SC-70-5, F.Cu at (21.8, 123.6)
- added U27: AP22913W6-7, footprint:SOT-23-6, F.Cu at (26.4, 122.1)
- added U28: DSPIC33EP512MU810-I/PT, footprint:TQFP-100-12x12, F.Cu at (222.9, 117.2)
- C44, C51, C71: value 1n -> 13p
- C68, C69: value 10n -> 1u; footprint footprint:CAP_NONPOL_0402 -> footprint:CAP_NONPOL_0805
- L1: value SRN8040-2R2Y -> PA5003.332NLT; footprint footprint:SRN8040 -> footprint:PA5003
- L2: value SRN8040-2R2Y -> PA5003.222NLT; footprint footprint:SRN8040 -> footprint:PA5003
- L3: value SRN8040-2R2Y -> PA5003.152NLT; footprint footprint:SRN8040 -> footprint:PA5003
- R65: value 10K -> 100K
- R67, R74: value 10K -> 22K1
- R69: value 3K24 -> 22K1
- R70: value 10K -> 124K
- R71: value 1K91 -> 10K
- R75: value 10K -> 30K1
- R81: value 30K1 -> 33K
- U10, U11, U9: value TLV62130ARGTR -> TPS54527DDAR; footprint footprint:VQFN-16-EP -> footprint:SO-8-150mil-EP
- U12: value TPS7A7002DDAR -> TPS7A7001DDAR
- moved MTG6 174.0 mm to (63.2, 51.1)
- moved MTG7 173.9 mm to (237.1, 126.7)
- moved R129 88.8 mm to (100.4, 148.1)
- moved R132 88.8 mm to (100.4, 155.3)
- moved R67 82.9 mm to (141.0, 150.2)
- moved U9 82.1 mm to (147.1, 149.8)
- moved R70 78.8 mm to (141.0, 152.3)
- moved R71 78.8 mm to (141.0, 154.4)
- moved R81 77.6 mm to (141.0, 156.6)
- moved HOLE1 75.6 mm to (63.2, 126.7)
- moved MTG5 75.6 mm to (63.2, 126.7)
- moved HOLE2 75.6 mm to (63.2, 51.1)
- moved MTG8 75.6 mm to (237.1, 51.1)
- moved L1 70.3 mm to (145.5, 143.8)
- moved R65 67.9 mm to (141.0, 148.2)
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Connections:
- net 1V0_CB renamed 1V05_CB
- C68 pad 1: Net-(U10-SS) -> GND
- C68 pad 2: GND -> Net-(U10-VREG)
- C69 pad 1: Net-(U11-SS) -> GND
- C69 pad 2: GND -> Net-(U11-VREG)
- C70 pad 1: Net-(U9-SS) -> GND
- C70 pad 2: GND -> Net-(U9-SS)
- D5 pad 1: Net-(D5-K) -> /Power Supply/PWR_LOG_EN
- D6 pad 1: Net-(D5-K) -> /Power Supply/PWR_LOG_EN
- D7 pad 2: Net-(D5-K) -> /Power Supply/PWR_LOG_EN
- L1 pad 1: Net-(L1-Pad1) -> Net-(U9-SW)
- L2 pad 1: Net-(L2-Pad1) -> Net-(U10-SW)
- L3 pad 1: Net-(L3-Pad1) -> Net-(U11-SW)
- R65 pad 2: Net-(D5-K) -> /Power Supply/PWR_LOG_EN
- R66 pad 2: Net-(U9-PG) -> Net-(Q13-D)
- R67 pad 1: Net-(U9-PG) -> Net-(U9-FB)
- R67 pad 2: 3V3_CB -> GND
- R71 pad 1: Net-(U9-FB) -> Net-(Q13-D)
- R71 pad 2: GND -> 3V3_CB
- R74 pad 1: Net-(U10-PG) -> Net-(U11-FB)
- R74 pad 2: 3V3_CB -> GND
- R83 pad 2: Net-(U11-PG) -> 1V8_CB
- U10 pad 1: Net-(L1-Pad1) -> /Power Supply/PWR_LOG_EN
- U10 pad 2: Net-(L1-Pad1) -> Net-(U10-FB)
- U10 pad 3: Net-(L1-Pad1) -> Net-(U10-VREG)
- U10 pad 4: Net-(U10-PG) -> Net-(U10-SS)
- U10 pad 5: Net-(U10-FB) -> GND
- U10 pad 6: GND -> Net-(U10-SW)
- U10 pad 7: GND -> Net-(U10-VBST)
- U10 pad 8: GND -> 12V0_CB
- U10 pad 9: Net-(U10-SS) -> GND
- U11 pad 1: Net-(L3-Pad1) -> /Power Supply/PWR_LOG_EN
- U11 pad 2: Net-(L3-Pad1) -> Net-(U11-FB)
- U11 pad 3: Net-(L3-Pad1) -> Net-(U11-VREG)
- U11 pad 4: Net-(U11-PG) -> Net-(U11-SS)
- U11 pad 5: Net-(U11-FB) -> GND
- U11 pad 6: GND -> Net-(U11-SW)
- U11 pad 7: GND -> Net-(U11-VBST)
- U11 pad 8: GND -> 12V0_CB
- U11 pad 9: Net-(U11-SS) -> GND
- U12 pad 2: Net-(U11-PG) -> 1V8_CB
- U9 pad 1: Net-(L2-Pad1) -> Net-(Q7-D)
- U9 pad 2: Net-(L2-Pad1) -> Net-(U9-FB)
- U9 pad 3: Net-(L2-Pad1) -> Net-(U9-VREG)
- U9 pad 4: Net-(U9-PG) -> Net-(U9-SS)
- U9 pad 5: Net-(U9-FB) -> GND
- U9 pad 6: GND -> Net-(U9-SW)
- U9 pad 7: GND -> Net-(U9-VBST)
- U9 pad 8: GND -> 12V0_CB
- U9 pad 9: Net-(U9-SS) -> GND
